Commit message: Model the real leg mechanism: 3 servos, 1:1 gear, parallelogram, foot four-bar
Fusion Fox_Prototype_03_v6_RL_Mechanism: 33 parts, 40 joints (hip / pivot / gear servo +
7 pins per leg, two closing loops), 4 pinion->gear motion links (12:12, reversed); saved
only after drive tests (gear = -pinion, shin || crank, Quad Link || femur, rear foot || femur).
MJCF fox.xml is the exact mechanism with 12 servo actuators; fox_reduced.xml and the URDF
are the tree with the servo map thigh = pivot, knee = -gear - pivot (foot = four-bar /
<mimic>). Knee limited at the loops' dead points. Isaac Lab FoxServoActuator takes servo
targets. MuJoCo + Isaac Sim checks pass; reduced tree matches the exact model to 0.04 mm.

Co-Authored-By: Claude Opus 5.5 <noreply@anthropic.com>

File: urdf/fox.urdf (robot description, URDF)
Before this commit: robot fox, 13 links, 12 joints
Links:
- added link FL_foot, mass 0.002518; collision mesh filename=../meshes/collision/FL_foot_reduced.stl; visual mesh filename=../meshes/visual/FL_foot_reduced.stl
- added link FR_foot, mass 0.002518; collision mesh filename=../meshes/collision/FR_foot_reduced.stl; visual mesh filename=../meshes/visual/FR_foot_reduced.stl
- added link RL_foot, mass 0.003072; collision mesh filename=../meshes/collision/RL_foot_reduced.stl; visual mesh filename=../meshes/visual/RL_foot_reduced.stl
- added link RR_foot, mass 0.003009; collision mesh filename=../meshes/collision/RR_foot_reduced.stl; visual mesh filename=../meshes/visual/RR_foot_reduced.stl
- link FL_calf: mass 0.010363 -> 0.007846; geometry collision mesh filename=../meshes/collision/FL_calf_reduced.stl; visual mesh filename=../meshes/visual/FL_calf_reduced.stl
- link FL_hip: mass 0.034795 -> 0.034433; geometry collision mesh filename=../meshes/collision/FL_hip_reduced.stl; visual mesh filename=../meshes/visual/FL_hip_reduced.stl
- link FL_thigh: mass 0.007137 -> 0.007500; geometry collision mesh filename=../meshes/collision/FL_thigh_reduced.stl; visual mesh filename=../meshes/visual/FL_thigh_reduced.stl
- link FR_calf: mass 0.010693 -> 0.008175; geometry collision mesh filename=../meshes/collision/FR_calf_reduced.stl; visual mesh filename=../meshes/visual/FR_calf_reduced.stl
- link FR_hip: mass 0.034796 -> 0.034433; geometry collision mesh filename=../meshes/collision/FR_hip_reduced.stl; visual mesh filename=../meshes/visual/FR_hip_reduced.stl
- link FR_thigh: mass 0.007137 -> 0.007500; geometry collision mesh filename=../meshes/collision/FR_thigh_reduced.stl; visual mesh filename=../meshes/visual/FR_thigh_reduced.stl
- link RL_calf: mass 0.010429 -> 0.007357; geometry collision mesh filename=../meshes/collision/RL_calf_reduced.stl; visual mesh filename=../meshes/visual/RL_calf_reduced.stl
- link RL_hip: mass 0.035295 -> 0.034933; geometry collision mesh filename=../meshes/collision/RL_hip_reduced.stl; visual mesh filename=../meshes/visual/RL_hip_reduced.stl
- link RL_thigh: mass 0.007402 -> 0.007764; geometry collision mesh filename=../meshes/collision/RL_thigh_reduced.stl; visual mesh filename=../meshes/visual/RL_thigh_reduced.stl
- link RR_calf: mass 0.009974 -> 0.006965; geometry collision mesh filename=../meshes/collision/RR_calf_reduced.stl; visual mesh filename=../meshes/visual/RR_calf_reduced.stl
- link RR_hip: mass 0.036785 -> 0.036423; geometry collision mesh filename=../meshes/collision/RR_hip_reduced.stl; visual mesh filename=../meshes/visual/RR_hip_reduced.stl
- link RR_thigh: mass 0.007311 -> 0.007674; geometry collision mesh filename=../meshes/collision/RR_thigh_reduced.stl; visual mesh filename=../meshes/visual/RR_thigh_reduced.stl
Joints:
- added joint FL_foot_joint: type revolute, parent FL_calf, child FL_foot, origin xyz=0.005365 0.002750 -0.067459 rpy=0 0 0, axis -0 1 0, limit lower=-3.1416 upper=3.1416 effort=10.000 velocity=50.00, mimic joint=FL_calf_joint multiplier=0.358775 offset=0
- added joint FR_foot_joint: type revolute, parent FR_calf, child FR_foot, origin xyz=0.005365 -0.002750 -0.067459 rpy=0 0 0, axis -0 1 0, limit lower=-3.1416 upper=3.1416 effort=10.000 velocity=50.00, mimic joint=FR_calf_joint multiplier=0.358775 offset=0
- added joint RL_foot_joint: type revolute, parent RL_calf, child RL_foot, origin xyz=-0.052566 0.001000 -0.053496 rpy=0 0 0, axis -0 1 0, limit lower=-3.1416 upper=3.1416 effort=10.000 velocity=50.00, mimic joint=RL_calf_joint multiplier=-1.000000 offset=0
- added joint RR_foot_joint: type revolute, parent RR_calf, child RR_foot, origin xyz=-0.052566 -0.001000 -0.053496 rpy=0 0 0, axis -0 1 0, limit lower=-3.1416 upper=3.1416 effort=10.000 velocity=50.00, mimic joint=RR_calf_joint multiplier=-1.000000 offset=0
- joint FL_calf_joint: origin xyz=-0.026270 0.001617 -0.070250 rpy=0 0 0 -> xyz=-0.026269 0.000000 -0.070249 rpy=0 0 0
- joint FL_hip_joint: origin xyz=0.071686 0.024238 0.007391 rpy=0 0 0 -> xyz=0.071686 0.024238 0.007390 rpy=0 0 0
- joint FL_thigh_joint: limit lower=-1.2000 upper=1.2000 effort=0.470 velocity=10.50 -> lower=-1.2000 upper=1.2000 effort=0.940 velocity=10.50; origin xyz=0.013074 0.018552 -0.002611 rpy=0 0 0 -> xyz=0.013073 0.017273 -0.002610 rpy=0 0 0
- joint FR_calf_joint: origin xyz=-0.026270 -0.001738 -0.070250 rpy=0 0 0 -> xyz=-0.026269 0.000000 -0.070249 rpy=0 0 0
- joint FR_hip_joint: origin xyz=0.071686 -0.024262 0.007391 rpy=0 0 0 -> xyz=0.071686 -0.024262 0.007390 rpy=0 0 0
- joint FR_thigh_joint: limit lower=-1.2000 upper=1.2000 effort=0.470 velocity=10.50 -> lower=-1.2000 upper=1.2000 effort=0.940 velocity=10.50; origin xyz=0.013074 -0.018528 -0.002611 rpy=0 0 0 -> xyz=0.013073 -0.017248 -0.002610 rpy=0 0 0
- joint RL_calf_joint: axis -0 1 -0 -> 0 1 0; limit lower=-1.2000 upper=1.2000 effort=0.470 velocity=10.50 -> lower=-1.2000 upper=0.7400 effort=0.470 velocity=10.50; origin xyz=0.038070 0.001795 -0.064620 rpy=0 0 0 -> xyz=0.038069 0.001750 -0.064620 rpy=0 0 0
- joint RL_hip_joint: origin xyz=-0.073606 0.024238 -0.000350 rpy=0 0 0 -> xyz=-0.073606 0.024238 -0.000351 rpy=0 0 0
- joint RL_thigh_joint: limit lower=-1.2000 upper=1.2000 effort=0.470 velocity=10.50 -> lower=-1.2000 upper=1.2000 effort=0.940 velocity=10.50; origin xyz=-0.012394 0.018550 -0.004430 rpy=0 0 0 -> xyz=-0.012394 0.017273 -0.004429 rpy=0 0 0
- joint RR_calf_joint: axis -0 1 -0 -> 0 1 0; limit lower=-1.2000 upper=1.2000 effort=0.470 velocity=10.50 -> lower=-1.2000 upper=0.7400 effort=0.470 velocity=10.50; origin xyz=0.038070 -0.001680 -0.064620 rpy=0 0 0 -> xyz=0.038069 -0.001500 -0.064620 rpy=0 0 0
- joint RR_hip_joint: origin xyz=-0.073382 -0.024238 -0.000187 rpy=0 0 0 -> xyz=-0.073382 -0.024238 -0.000188 rpy=0 0 0
- joint RR_thigh_joint: limit lower=-1.2000 upper=1.2000 effort=0.470 velocity=10.50 -> lower=-1.2000 upper=1.2000 effort=0.940 velocity=10.50; origin xyz=-0.012618 -0.018531 -0.004593 rpy=0 0 0 -> xyz=-0.012618 -0.017522 -0.004593 rpy=0 0 0
