Commit message: v7 sim model without the rear hip spacer
The robot will be built without the spacer (no longer screws), so v7/ now models v6 geometry with the v7 drive:
tools/raw_v7_without_spacer.py makes raw_v7_nospacer/ from the v6 export (base, legs, all joints) plus the v7
gear and pinion links moved back to their v6 positions (mass/inertia moved with them), the 2:1 motion links
and the v7 pinion range; build_robot.py --raw raw_v7_nospacer --out v7.
Stance: front feet 25.5 mm ahead of the hips, rear 34.1 mm behind; worst servo 40 % of stall (trot estimate,
34 % with the spacer, 72 % v6); standing in MuJoCo 11 %. All MuJoCo checks pass. The spacer build's Fusion
evidence moved to v7/validation/cad/.

Co-Authored-By: Claude Opus 5.5 <noreply@anthropic.com>

File: v7/urdf/fox.urdf (robot description, URDF)
Before this commit: robot fox, 17 links, 16 joints
Links:
- link base: mass 0.335624 -> 0.330454
Joints:
- joint FL_hip_joint: origin xyz=0.071686 0.024238 -0.002007 rpy=0 0 0 -> xyz=0.071686 0.024238 0.007390 rpy=0 0 0
- joint FL_thigh_joint: axis 0 1 -0 -> 0 1 0
- joint FR_hip_joint: origin xyz=0.071686 -0.024262 -0.002007 rpy=0 0 0 -> xyz=0.071686 -0.024262 0.007390 rpy=0 0 0
- joint FR_thigh_joint: axis 0 1 -0 -> 0 1 0
- joint RL_calf_joint: origin xyz=0.038068 0.001750 -0.064620 rpy=0 0 0 -> xyz=0.038069 0.001750 -0.064620 rpy=0 0 0
- joint RL_hip_joint: axis 0.939693 -0 0.34202 -> 0.939693 0 0.34202; origin xyz=-0.080446 0.024238 0.009046 rpy=0 0 0 -> xyz=-0.073606 0.024238 -0.000351 rpy=0 0 0
- joint RR_hip_joint: axis 0.939693 -0 0.34202 -> 0.939693 0 0.34202; origin xyz=-0.080223 -0.024238 0.009209 rpy=0 0 0 -> xyz=-0.073382 -0.024238 -0.000188 rpy=0 0 0
- joint RR_thigh_joint: origin xyz=-0.012617 -0.017522 -0.004592 rpy=0 0 0 -> xyz=-0.012618 -0.017522 -0.004593 rpy=0 0 0
